File: PCB Files/micromouse V2.kicad_sch (KiCad schematic)
At the start: 59 parts, among them J1 TOF1, J2 TOF1, J3 Conn_02x02_Counter_Clockwise, J4 BATT, J5 TOF1, J6 Conn_01x02_Pin, J7 Motor 1, J8 Motor 2, J9 USB-C, SW1 BOOT0, SW2 BOOT1, SW3 A, SW4 B, SW5 C, SW6 RESET, SW7 POWER, U1 L7806, U2 AMS1117-3.3, U3 L7805, U4 STM32F103C8Tx, U5 SSD1306, U6 TB6612FNG, X1 SG-3030CM, Y1 8MHz, Y2 32.768K

Commit message: Fixed PCB Layout
Parts:
- removed SW4: B, Button_Switch_THT:SW_PUSH_6mm_H13mm, symbol Switch:SW_Push
- removed X1: SG-3030CM, Oscillator:Oscillator_SMD_SeikoEpson_SG3030CM, symbol Oscillator:SG-3030CM
- added C15, C16, C17: 0.1uF, Capacitor_SMD:C_0805_2012Metric_Pad1.18x1.45mm_HandSolder, symbol Device:C
- added R7, R8, R9: 10K, Resistor_SMD:R_0805_2012Metric_Pad1.20x1.40mm_HandSolder, symbol Device:R
- added SW6: C, Button_Switch_THT:SW_PUSH_6mm_H13mm, symbol Switch:SW_Push
- SW5: value C -> B
- Y1: footprint Crystal:Crystal_HC49-4H_Vertical -> Custom:Crystal_ABLS2-8.000MHZ-D4Y-T
- Y2: footprint Custom:Crystal_ABLS2-8.000MHZ-D4Y-T -> Custom:XTAL_ABS07-32.768KHZ-T
- renumbered C17 to C18, C15 to C19, C16 to C20, C18 to C21, C19 to C22, R6 to R10, R7 to R11, R8 to R5, R5 to R6, SW7 to SW3, SW3 to SW4, SW6 to SW7
Connections:
- net +3.3V: now also R3.1, SW4.2, SW5.2, C15.1, C16.1, C17.1, SW6.2; no longer D1.2 (A)
- net GND: now also D1.1 (K), R7.2, R8.2, R9.2; no longer R3.2, SW4.1, SW5.1
- net SW1: now also SW4.1, C15.2, R7.1; no longer SW4.2
- net SW2: now also SW5.1, C16.2, R8.1
- net SW3: now also C17.2, R9.1, SW6.1; no longer SW5.2
- new net: D1.2 (A), R3.2
Other:
- moved on the sheet: C18, C19, C20, C21, C22, D1, D4, D5, D6, J9, R10, R11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

Commit message: default
Parts:
- added C23: 10nF, Capacitor_SMD:C_0805_2012Metric, symbol Device:C
- added C24, C25: 100nF, Capacitor_SMD:C_0805_2012Metric, symbol Device:C
- added C26: 2.2nF, Capacitor_SMD:C_0805_2012Metric, symbol Device:C
- added D7: GYRO, LED_SMD:LED_0805_2012Metric, symbol Device:LED
- added R12, R13, R14: 4.7K, Resistor_SMD:R_0805_2012Metric, symbol Device:R
- added R15: 47R, Resistor_SMD:R_0805_2012Metric, symbol Device:R
- added U7: MPU-6050, Sensor_Motion:InvenSense_QFN-24_4x4mm_P0.5mm, symbol Sensor_Motion:MPU-6050
- C1: footprint Capacitor_SMD:C_0805_2012Metric_Pad1.18x1.45mm_HandSolder -> Capacitor_SMD:C_0805_2012Metric; JLCPCB Part# (none) -> C1713
- C10, C9: footprint Capacitor_SMD:C_0805_2012Metric_Pad1.18x1.45mm_HandSolder -> Capacitor_SMD:C_0805_2012Metric; JLCPCB Part# (none) -> C95841
- C11, C13: footprint Capacitor_SMD:C_0805_2012Metric_Pad1.18x1.45mm_HandSolder -> Capacitor_SMD:C_0805_2012Metric; JLCPCB Part# (none) -> C318723
- C12, C14, C2, C3, C4, C5: footprint Capacitor_SMD:C_0805_2012Metric_Pad1.18x1.45mm_HandSolder -> Capacitor_SMD:C_0805_2012Metric; JLCPCB Part# (none) -> C520082
- C15, C16, C17: value 0.1uF -> 100nF; footprint Capacitor_SMD:C_0805_2012Metric_Pad1.18x1.45mm_HandSolder -> Capacitor_SMD:C_0805_2012Metric; JLCPCB Part# (none) -> C520082
- C18, C7, C8: footprint Capacitor_SMD:C_0805_2012Metric_Pad1.18x1.45mm_HandSolder -> Capacitor_SMD:C_0805_2012Metric; JLCPCB Part# (none) -> C24123
- C19, C20, C21, C22: footprint Capacitor_SMD:C_0805_2012Metric_Pad1.18x1.45mm_HandSolder -> Capacitor_SMD:C_0805_2012Metric; JLCPCB Part# (none) -> C1798
- C6: footprint Capacitor_SMD:C_0805_2012Metric_Pad1.18x1.45mm_HandSolder -> Capacitor_SMD:C_0805_2012Metric; JLCPCB Part# (none) -> C519909
- D1, D2, D3, D4, D5: footprint LED_SMD:LED_0805_2012Metric_Pad1.15x1.40mm_HandSolder -> LED_SMD:LED_0805_2012Metric; JLCPCB Part# (none) -> C2297
- D6: JLCPCB Part# (none) -> C7074
- FB1: JLCPCB Part# (none) -> C88990
- J4: JLCPCB Part# (none) -> C265283
- J7, J8: JLCPCB Part# (none) -> C265366
- J9: JLCPCB Part# (none) -> C165948
- R1: footprint Resistor_SMD:R_0805_2012Metric_Pad1.20x1.40mm_HandSolder -> Resistor_SMD:R_0805_2012Metric; JLCPCB Part# (none) -> C17630
- R10: footprint Resistor_SMD:R_0805_2012Metric_Pad1.20x1.40mm_HandSolder -> Resistor_SMD:R_0805_2012Metric; JLCPCB Part# (none) -> C17557
- R11: footprint Resistor_SMD:R_0805_2012Metric_Pad1.20x1.40mm_HandSolder -> Resistor_SMD:R_0805_2012Metric; JLCPCB Part# (none) -> C17423
- R2: footprint Resistor_SMD:R_0805_2012Metric_Pad1.20x1.40mm_HandSolder -> Resistor_SMD:R_0805_2012Metric; JLCPCB Part# (none) -> C17802
- R3, R6: footprint Resistor_SMD:R_0805_2012Metric_Pad1.20x1.40mm_HandSolder -> Resistor_SMD:R_0805_2012Metric; JLCPCB Part# (none) -> C17714
- R4, R7, R8, R9: footprint Resistor_SMD:R_0805_2012Metric_Pad1.20x1.40mm_HandSolder -> Resistor_SMD:R_0805_2012Metric; JLCPCB Part# (none) -> C17414
- R5: footprint Resistor_SMD:R_0805_2012Metric_Pad1.20x1.40mm_HandSolder -> Resistor_SMD:R_0805_2012Metric; JLCPCB Part# (none) -> C17514
- SW1, SW2, SW3: footprint Button_Switch_THT:SW_Slide_SPDT_Straight_CK_OS102011MS2Q -> Custom:SW_SS12D07VG4; JLCPCB Part# (none) -> C2939726
- SW4, SW5, SW6, SW7: JLCPCB Part# (none) -> C7470131
- U2: JLCPCB Part# (none) -> C6186
- U4: JLCPCB Part# (none) -> C8734
- U6: JLCPCB Part# (none) -> C141517
- Y1: JLCPCB Part# (none) -> C596832
- Y2: JLCPCB Part# (none) -> C130253
Connections:
- net +3.3V: now also C23.1, C24.1, R12.2, R13.2, R15.1, U7.13 (VDD), U7.8 (VLOGIC)
- net GND: now also C23.2, C24.2, C25.1, C26.2, D7.1 (K), R14.1, U7.1 (CLKIN), U7.11 (FSYNC), U7.18 (GND)
- net SCL2: now also R13.1, U7.23 (SCL)
- net SDA2: now also R12.1, U7.24 (SDA)
- net OSC32_IN renamed LSE_IN
- net OSC32_OUT renamed LSE_OUT
- new net: D7.2 (A), R15.2
- new net: C25.2, U7.10 (REGOUT)
- new net: C26.1, U7.20 (CPOUT)
- new net: R14.2, U7.9 (AD0)
- new net GYRO_INT: U7.12 (INT)
- no-connect marks 16 -> 18
Other:
- note added: "MPU-6050"
