File: PCB Files/micromouse V2.kicad_pcb (KiCad board)
At the start: 2 copper layers, 100 x 130 mm, 78 parts, among them J1 TOF1, J2 TOF1, J3 Conn_02x02_Counter_Clockwise, J4 BATT, J5 TOF1, J6 Conn_01x02_Pin, J7 Motor 1, J8 Motor 2, J9 USB-C, SW1 BOOT0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

Commit message: Default
Other:
- board text removed: "MININDU PASAN"
